Commit message: build logs, experimenting with files

File: install/auv_description/share/auv_description/model/auv.xacro (robot description, xacro)
@@ -1,7 +1,9 @@
 <?xml version="1.0"?>
 <robot xmlns:xacro="http://www.ros.org/wiki/xacro" name="auv">
+  <!-- settings -->
+  <xacro:property name="imuHz" value="100.0"/>
   <!-- var -->
   <xacro:property name="cwd" value="/home/ubuntu/dev_ws/src/auv_description/model"/>
-  <xacro:property name="PI" value="3.1415926535897931"/>
+  <xacro:property name="pi" value="3.1415926535897931"/>
   <!-- incl -->
   <xacro:include filename="${cwd}/materials.xacro" />
@@ -97,5 +99,5 @@
     <sensor name="imu_sensor" type="imu">
       <always_on>1</always_on>
-      <update_rate>1</update_rate>
+      <update_rate>${imuHz}</update_rate>
       <visualize>true</visualize>
       <topic>imu</topic>
