Commit message: update

File: install/auv_description/share/auv_description/model/auv.urdf (robot description, URDF)
Before this commit: robot test, 3 links, 2 joints
Links:
- added link caster_link, mass 1; collision sphere radius=0.2; visual sphere radius=0.2
- added link dummy
Joints:
- added joint caster_joint: type fixed, parent base_link, child caster_link, origin xyz=-0.8 0 -0.2 rpy=0 0 0
- added joint dummy_joint: type fixed, parent dummy, child base_link

File: install/auv_description/share/auv_description/model/auv.xacro (robot description, xacro)
@@ -1,10 +1,13 @@
 <?xml version="1.0"?>
-<robot xmlns:xacro="http://www.ros.org/wiki/xacro" name="test">
+<robot xmlns:xacro="http://www.ros.org/wiki/xacro" name="auv">
   <!-- var -->
-  <xacro:property name="cwd" value="/home/ubuntu/urdf"/>
+  <xacro:property name="cwd" value="/home/ubuntu/dev_ws/src/auv_description/model"/>
   <xacro:property name="PI" value="3.1415926535897931"/>
   <!-- incl -->
   <xacro:include filename="${cwd}/materials.xacro" />
+  <xacro:include filename="${cwd}/inertial_macros.xacro" />
   <!-- base -->
+  <link name="dummy">
+  </link>
   <link name="base_link">
     <inertial>
@@ -23,4 +26,8 @@
     </collision>
   </link>
+  <joint name="dummy_joint" type="fixed">
+     <parent link="dummy"/>
+     <child link="base_link"/>
+  </joint>
   <gazebo reference='base_link'>
     <xacro:red/>
@@ -54,46 +61,24 @@
   <xacro:wheel name="fr" x="0.5" y="0.6"/>
   <!-- caster -->
-  <gazebo>
-    <frame name="caster_frame" attached_to='base_link'>
-      <pose>-0.8 0 -0.2 0 0 0</pose>
-    </frame>
-    <link name='caster_link'>
-      <pose relative_to='caster_frame'/>
-      <inertial>
-          <mass>1</mass>
-          <inertia>
-              <ixx>0.016</ixx>
-              <ixy>0</ixy>
-              <ixz>0</ixz>
-              <iyy>0.016</iyy>
-              <iyz>0</iyz>
-              <izz>0.016</izz>
-          </inertia>
-      </inertial>
-      <visual name="visual">
-          <geometry>
-              <sphere>
-                  <radius>0.2</radius>
-              </sphere>
-          </geometry>
-          <material>
-              <ambient>0.0 1 0.0 1</ambient>
-              <diffuse>0.0 1 0.0 1</diffuse>
-              <specular>0.0 1 0.0 1</specular>
-          </material>
-      </visual>
-      <collision name="collision">
-          <geometry>
-              <sphere>
-                  <radius>0.2</radius>
-              </sphere>
-          </geometry>
-      </collision>
-    </link>
-    <joint name='caster_joint' type='ball'>
-      <parent>base_link</parent>
-      <child>caster_link</child>
-    </joint>
-  </gazebo>
+  <link name="caster_link">
+    <xacro:inertial_sphere mass="0.1" radius="0.2">
+      <origin xyz="0 0 0" rpy="0 0 0"/>
+    </xacro:inertial_sphere>
+    <visual>
+      <geometry>
+        <sphere radius="0.2"/>
+      </geometry>
+    </visual>
+    <collision>
+      <geometry>
+        <sphere radius="0.2"/>
+      </geometry>
+    </collision>
+  </link>
+  <joint name="caster_joint" type="fixed">
+    <origin xyz="-0.8 0 -0.2" rpy="0 0 0"/>
+    <parent link="base_link"/>
+    <child link="caster_link"/>
+  </joint>
   <!-- plugins -->
   <gazebo>

Commit message: First working version!

File: install/auv_description/share/auv_description/model/auv.urdf (robot description, URDF)
Before this commit: robot auv, 5 links, 4 joints
Links:
- link caster_link: mass 1 -> 1e-06

File: install/auv_description/share/auv_description/model/auv.xacro (robot description, xacro)
@@ -62,5 +62,5 @@
   <!-- caster -->
   <link name="caster_link">
-    <xacro:inertial_sphere mass="0.1" radius="0.2">
+    <xacro:inertial_sphere mass="0.000001" radius="0.2">
       <origin xyz="0 0 0" rpy="0 0 0"/>
     </xacro:inertial_sphere>

Commit message: imu_corrector part1, default.rviz

File: install/auv_description/share/auv_description/model/auv.urdf (robot description, URDF)
Before this commit: robot auv, 5 links, 4 joints
Links:
- removed link dummy
- added link dummy_link
Joints:
- joint dummy_joint: parent dummy -> dummy_link

File: install/auv_description/share/auv_description/model/auv.xacro (robot description, xacro)
@@ -1,106 +1 @@
-<?xml version="1.0"?>
-<robot xmlns:xacro="http://www.ros.org/wiki/xacro" name="auv">
-  <!-- settings -->
-  <xacro:property name="imuHz" value="100.0"/>
-  <!-- var -->
-  <xacro:property name="cwd" value="/home/ubuntu/dev_ws/src/auv_description/model"/>
-  <xacro:property name="pi" value="3.1415926535897931"/>
-  <!-- incl -->
-  <xacro:include filename="${cwd}/materials.xacro" />
-  <xacro:include filename="${cwd}/inertial_macros.xacro" />
-  <!-- base -->
-  <link name="dummy">
-  </link>
-  <link name="base_link">
-    <inertial>
-        <mass value="1.14395"/>
-        <inertia ixx="0.095329" ixy="0" ixz="0" iyy="0.381317" iyz="0" izz="0.476646"/>
-    </inertial>
-    <visual>
-      <geometry>
-        <box size="2.0 1.0 0.5"/>
-      </geometry>
-    </visual>
-    <collision>
-      <geometry>
-        <box size="2.0 1.0 0.5"/>
-      </geometry>
-    </collision>
-  </link>
-  <joint name="dummy_joint" type="fixed">
-     <parent link="dummy"/>
-     <child link="base_link"/>
-  </joint>
-  <gazebo reference='base_link'>
-    <xacro:red/>
-  </gazebo>
-  <!-- driving wheels -->
-  <xacro:macro name="wheel" params="name x y">
-    <link name="${name}_link">
-      <inertial>
-        <mass value="1"/>
-        <inertia ixx="0.043333" ixy="0" ixz="0" iyy="0.043333" iyz="0" izz="0.08"/>
-      </inertial>
-      <visual>
-        <geometry>
-          <cylinder radius="0.4" length="0.2"/>
-        </geometry>
-      </visual>
-      <collision>
-        <geometry>
-          <cylinder radius="0.4" length="0.2"/>
-        </geometry>
-      </collision>
-    </link>
-    <joint name="${name}_joint" type="continuous">
-      <origin xyz="${x} ${y} 0.0" rpy="1.5707 0.0 0.0"/>
-      <parent link="base_link"/>
-      <child link="${name}_link"/>
-      <axis xyz="0.0 0.0 1.0"/>
-    </joint>
-  </xacro:macro>
-  <xacro:wheel name="fl" x="0.5" y="-0.6"/>
-  <xacro:wheel name="fr" x="0.5" y="0.6"/>
-  <!-- caster -->
-  <link name="caster_link">
-    <xacro:inertial_sphere mass="0.000001" radius="0.2">
-      <origin xyz="0 0 0" rpy="0 0 0"/>
-    </xacro:inertial_sphere>
-    <visual>
-      <geometry>
-        <sphere radius="0.2"/>
-      </geometry>
-    </visual>
-    <collision>
-      <geometry>
-        <sphere radius="0.2"/>
-      </geometry>
-    </collision>
-  </link>
-  <joint name="caster_joint" type="fixed">
-    <origin xyz="-0.8 0 -0.2" rpy="0 0 0"/>
-    <parent link="base_link"/>
-    <child link="caster_link"/>
-  </joint>
-  <!-- plugins -->
-  <gazebo>
-    <plugin
-      filename="ignition-gazebo-diff-drive-system"
-      name="ignition::gazebo::systems::DiffDrive">
-      <left_joint>fl_joint</left_joint>
-      <right_joint>fr_joint</right_joint>
-      <wheel_separation>1</wheel_separation>
-      <wheel_radius>0.4</wheel_radius>
-      <odom_publish_frequency>1</odom_publish_frequency>
-      <topic>cmd_vel</topic>
-    </plugin>
-  </gazebo>
-  <gazebo reference="base_link">
-    <sensor name="imu_sensor" type="imu">
-      <always_on>1</always_on>
-      <update_rate>${imuHz}</update_rate>
-      <visualize>true</visualize>
-      <topic>imu</topic>
-    </sensor>
-  </gazebo>
-</robot>
+/home/ubuntu/dev_ws/src/auv_description/model/auv.xacro

File: install/auv_description/share/auv_description/model/inertial_macros.xacro (robot description, xacro)
@@ -1,31 +1 @@
-<?xml version="1.0"?>
-<robot xmlns:xacro="http://www.ros.org/wiki/xacro" >
-    <!-- Specify some standard inertial calculations https://en.wikipedia.org/wiki/List_of_moments_of_inertia -->
-    <xacro:macro name="inertial_sphere" params="mass radius *origin">
-        <inertial>
-            <xacro:insert_block name="origin"/>
-            <mass value="${mass}" />
-            <inertia ixx="${(2/5) * mass * (radius*radius)}" ixy="0.0" ixz="0.0"
-                    iyy="${(2/5) * mass * (radius*radius)}" iyz="0.0"
-                    izz="${(2/5) * mass * (radius*radius)}" />
-        </inertial>
-    </xacro:macro>
-    <xacro:macro name="inertial_box" params="mass x y z *origin">
-        <inertial>
-            <xacro:insert_block name="origin"/>
-            <mass value="${mass}" />
-            <inertia ixx="${(1/12) * mass * (y*y+z*z)}" ixy="0.0" ixz="0.0"
-                    iyy="${(1/12) * mass * (x*x+z*z)}" iyz="0.0"
-                    izz="${(1/12) * mass * (x*x+y*y)}" />
-        </inertial>
-    </xacro:macro>
-    <xacro:macro name="inertial_cylinder" params="mass length radius *origin">
-        <inertial>
-            <xacro:insert_block name="origin"/>
-            <mass value="${mass}" />
-            <inertia ixx="${(1/12) * mass * (3*radius*radius + length*length)}" ixy="0.0" ixz="0.0"
-                    iyy="${(1/12) * mass * (3*radius*radius + length*length)}" iyz="0.0"
-                    izz="${(1/2) * mass * (radius*radius)}" />
-        </inertial>
-    </xacro:macro>
-</robot>
+/home/ubuntu/dev_ws/src/auv_description/model/inertial_macros.xacro

File: install/auv_description/share/auv_description/model/materials.xacro (robot description, xacro)
@@ -1,21 +1 @@
-<?xml version="1.0"?>
-<robot xmlns:xacro="http://www.ros.org/wiki/xacro" name="materials">
-  <xacro:macro name="color" params="r g b">
-  	<visual>
-      <material>
-      	<ambient>${r} ${g} ${b} 1</ambient>
-        <diffuse>${r} ${g} ${b} 1</diffuse>
-        <specular>${r} ${g} ${b} 1</specular>
-      </material>
-    </visual>
-  </xacro:macro>
-	<xacro:macro name="red">
-		<xacro:color r="1" g="0" b="0"/>
-	</xacro:macro>
-	<xacro:macro name="green">
-		<xacro:color r="0" g="1" b="0"/>
-	</xacro:macro>
-	<xacro:macro name="blue">
-		<xacro:color r="0" g="0" b="1"/>
-	</xacro:macro>
-</robot>
+/home/ubuntu/dev_ws/src/auv_description/model/materials.xacro

File: src/auv_description/model/auv.xacro (robot description, xacro)
@@ -6,9 +6,10 @@
   <xacro:property name="cwd" value="/home/ubuntu/dev_ws/src/auv_description/model"/>
   <xacro:property name="pi" value="3.1415926535897931"/>
+  <xacro:property name="dummy_link_name" value="dummy"/>
   <!-- incl -->
   <xacro:include filename="${cwd}/materials.xacro" />
   <xacro:include filename="${cwd}/inertial_macros.xacro" />
   <!-- base -->
-  <link name="dummy">
+  <link name="${dummy_link_name}">
   </link>
   <link name="base_link">
@@ -29,5 +30,5 @@
   </link>
   <joint name="dummy_joint" type="fixed">
-     <parent link="dummy"/>
+     <parent link="${dummy_link_name}"/>
      <child link="base_link"/>
   </joint>
@@ -102,4 +103,15 @@
       <visualize>true</visualize>
       <topic>imu</topic>
+      <angular_velocity>
+        <x><noise type="none"/></x>
+        <y><noise type="none"/></y>
+        <z><noise type="none"/></z>
+      </angular_velocity>
+      <linear_acceleration>
+        <x><noise type="none"/></x>
+        <y><noise type="none"/></y>
+        <z><noise type="none"/></z>
+      </linear_acceleration>
+      <gaussian_noise>0.0</gaussian_noise>
     </sensor>
   </gazebo>

Commit message: update

File: install/auv_description/share/auv_description/model/auv.urdf (robot description, URDF)
Before this commit: robot auv, 5 links, 4 joints
Links:
- removed link dummy_link
- added link dummy
Joints:
- joint dummy_joint: parent dummy_link -> dummy
