Commit message: robot localization working, added sam_bot for testing

File: src/robot_description/model/rover.xacro (robot description, xacro)
@@ -29,5 +29,5 @@
     <xacro:cylinder_link name="${name}_link" mass="1.2" radius="${WHEEL_RADIUS}" length="${WHEEL_LEN}"/>
     <joint name="${name}_joint" type="continuous">
-      <origin xyz="${x} ${y} 0.0" rpy="${PI/2} 0.0 0.0"/>
+      <origin xyz="${x} ${y} 0.0" rpy="${PI/2} ${PI} ${PI}"/>
       <parent link="base_link"/>
       <child link="${name}_link"/>

Commit message: Working version: ekf, odom, imu, etc

File: src/robot_description/model/rover.xacro (robot description, xacro)
@@ -3,8 +3,10 @@
   <!-- settings -->
   <xacro:property name="IMU_HZ" value="100.0"/>
+  <xacro:property name="ODOM_HZ" value="100.0"/>
   <xacro:property name="POSE_HZ" value="100.0"/>
   <xacro:property name="WHEEL_RADIUS" value="0.3"/>
-  <xacro:property name="WHEEL_LEN" value="0.3"/>
-  <xacro:property name="SZ" value="1.0"/>
+  <xacro:property name="WHEEL_THICKNESS" value="0.3"/>
+  <xacro:property name="LEN" value="2.0"/>
+  <xacro:property name="WIDTH" value="1.0"/>
   <!-- const -->
   <xacro:property name="CWD" value="/home/ubuntu/dev_ws/src/robot_description"/>
@@ -17,5 +19,5 @@
   <link name="${DUMMY_LINK_NAME}"/>
   <!-- base -->
-  <xacro:box_link name="base_link" mass="2" x="${SZ}" y="${SZ}" z="${SZ/2}"/>
+  <xacro:box_link name="base_link" mass="2" x="${LEN}" y="${WIDTH}" z="${WHEEL_RADIUS}"/>
   <joint name="dummy_joint" type="fixed">
      <parent link="${DUMMY_LINK_NAME}"/>
@@ -27,5 +29,5 @@
   <!-- wheels -->
   <xacro:macro name="wheel" params="name x y">
-    <xacro:cylinder_link name="${name}_link" mass="1.2" radius="${WHEEL_RADIUS}" length="${WHEEL_LEN}"/>
+    <xacro:cylinder_link name="${name}_link" mass="1.2" radius="${WHEEL_RADIUS}" length="${WHEEL_THICKNESS}"/>
     <joint name="${name}_joint" type="continuous">
       <origin xyz="${x} ${y} 0.0" rpy="${PI/2} ${PI} ${PI}"/>
@@ -35,7 +37,17 @@
     </joint>
   </xacro:macro>
-  <xacro:wheel name="fl" x="0" y="0.6"/>
-  <xacro:wheel name="fr" x="0" y="-0.6"/>
+  <xacro:wheel name="fl" x="${LEN/2-WHEEL_RADIUS}" y="${WIDTH/2+WHEEL_THICKNESS/2}"/>
+  <xacro:wheel name="fr" x="${LEN/2-WHEEL_RADIUS}" y="${-WIDTH/2-WHEEL_THICKNESS/2}"/>
   <!-- caster -->
+  <xacro:sphere_link name="caster_link" mass="1.2" radius="${WHEEL_RADIUS}"/>
+  <joint name="caster_joint" type="fixed">
+      <origin xyz="${-LEN/2+WHEEL_RADIUS} 0 0" rpy="0 0 0"/>
+      <parent link="base_link"/>
+      <child link="caster_link"/>
+  </joint>
+  <gazebo reference="caster_link">
+    <mu1>0</mu1>
+    <mu2>0</mu2>
+  </gazebo>
   <!-- plugins -->
   <gazebo>
@@ -45,7 +57,7 @@
       <left_joint>fl_joint</left_joint>
       <right_joint>fr_joint</right_joint>
-      <wheel_separation>1</wheel_separation>
+      <wheel_separation>${WIDTH}</wheel_separation>
       <wheel_radius>${WHEEL_RADIUS}</wheel_radius>
-      <odom_publish_frequency>${IMU_HZ}</odom_publish_frequency>
+      <odom_publish_frequency>${ODOM_HZ}</odom_publish_frequency>
       <topic>cmd_vel</topic>
     </plugin>

File: src/robot_description/utils/basic_links.xacro (robot description, xacro)
@@ -30,4 +30,21 @@
     </xacro:macro>
     <!-- Basic link macros -->
+    <xacro:macro name="sphere_link" params="name mass radius">
+        <link name="${name}">
+            <xacro:inertial_sphere mass="${mass}" radius="${radius}">
+                <origin xyz="0 0 0" rpy="0 0 0"/>
+            </xacro:inertial_sphere>
+            <visual>
+                <geometry>
+                    <sphere radius="${radius}"/>
+                </geometry>
+            </visual>
+            <collision>
+                <geometry>
+                    <sphere radius="${radius}"/>
+                </geometry>
+            </collision>
+        </link>
+    </xacro:macro>
     <xacro:macro name="box_link" params="name mass x y z">
         <link name="${name}">

Commit message: odometer plugin works now!

File: src/robot_description/model/rover.xacro (robot description, xacro)
@@ -1,7 +1,8 @@
-<?xml version="1.0"?>
-<robot xmlns:xacro="http://www.ros.org/wiki/xacro" name="rover">
+<?xml version="1.0" ?>
+<robot xmlns:xacro="http://www.ros.org/wiki/xacro" xmlns:ignition="http://www.ros.org/wiki/xacro" name="rover">
   <!-- settings -->
   <xacro:property name="IMU_HZ" value="100.0"/>
   <xacro:property name="ODOM_HZ" value="100.0"/>
+  <xacro:property name="ODOMETER_HZ" value="1.0"/>
   <xacro:property name="POSE_HZ" value="100.0"/>
   <xacro:property name="WHEEL_RADIUS" value="0.3"/>
@@ -91,3 +92,16 @@
     </sensor>
   </gazebo>
+  <gazebo reference="base_link">
+    <sensor name="LUCAS_ODOMETER" type="custom" ignition:type="odometer">
+      <always_on>1</always_on>
+      <update_rate>30</update_rate>
+      <visualize>true</visualize>
+      <ignition:odometer>
+        <noise type="gaussian">
+          <mean>0.00001</mean>
+          <stddev>0.00001</stddev>
+        </noise>
+      </ignition:odometer>
+    </sensor>
+  </gazebo>
 </robot>
